Commit message: set up simulation of rrbot using flawed internal model in rviz

File: rrbot_description/urdf/broken.xacro (robot description, xacro)
@@ -1,10 +1,10 @@
 <?xml version="1.0"?>
 <!-- Revolute-Revolute Manipulator -->
-<robot name="rrbot" xmlns:xacro="http://www.ros.org/wiki/xacro">
+<robot name="broken" xmlns:xacro="http://www.ros.org/wiki/xacro">
   <!-- Constants for robot dimensions -->
   <xacro:property name="PI" value="3.1415926535897931"/>
   <xacro:property name="mass" value="1" /> <!-- arbitrary value for mass -->
   <xacro:property name="width" value="0.1" /> <!-- Square dimensions (widthxwidth) of beams -->
-  <xacro:property name="height1" value="2" /> <!-- Link 1 -->
+  <xacro:property name="height1" value="1.9" /> <!-- Link 1 -->
   <xacro:property name="height2" value="1" /> <!-- Link 2 -->
   <xacro:property name="height3" value="1" /> <!-- Link 3 -->

Commit message: Setup launch files so that the two simulation will share the same control

File: rrbot_description/urdf/broken.xacro (robot description, xacro)
@@ -26,5 +26,5 @@
       <origin xyz="0 0 ${height1/2}" rpy="0 0 0"/>
       <geometry>
-	<box size="${width} ${width} ${height1}"/>
+	     <box size="${width} ${width} ${height1}"/>
       </geometry>
     </collision>
@@ -32,7 +32,7 @@
       <origin xyz="0 0 ${height1/2}" rpy="0 0 0"/>
       <geometry>
-	<box size="${width} ${width} ${height1}"/>
+	     <box size="${width} ${width} ${height1}"/>
       </geometry>
-      <material name="orange"/>
+      <material name="black"/>
     </visual>
     <inertial>
@@ -57,5 +57,5 @@
       <origin xyz="0 0 ${height2/2 - axel_offset}" rpy="0 0 0"/>
       <geometry>
-	<box size="${width} ${width} ${height2}"/>
+	     <box size="${width} ${width} ${height2}"/>
       </geometry>
     </collision>
@@ -63,5 +63,5 @@
       <origin xyz="0 0 ${height2/2 - axel_offset}" rpy="0 0 0"/>
       <geometry>
-	<box size="${width} ${width} ${height2}"/>
+	     <box size="${width} ${width} ${height2}"/>
       </geometry>
       <material name="black"/>
@@ -88,5 +88,5 @@
       <origin xyz="0 0 ${height3/2 - axel_offset}" rpy="0 0 0"/>
       <geometry>
-	<box size="${width} ${width} ${height3}"/>
+	     <box size="${width} ${width} ${height3}"/>
       </geometry>
     </collision>
@@ -94,7 +94,7 @@
       <origin xyz="0 0 ${height3/2 - axel_offset}" rpy="0 0 0"/>
       <geometry>
-	<box size="${width} ${width} ${height3}"/>
+	     <box size="${width} ${width} ${height3}"/>
       </geometry>
-      <material name="orange"/>
+      <material name="black"/>
     </visual>
     <inertial>
@@ -118,5 +118,5 @@
       <origin xyz="0 0 0" rpy="0 0 0"/>
       <geometry>
-	<box size="0.1 0.1 0.1"/>
+	     <box size="0.1 0.1 0.1"/>
       </geometry>
     </collision>
@@ -134,5 +134,5 @@
   </link>
   <joint name="camera_joint" type="fixed">
-    <origin xyz="0 2 1" rpy="0 0 ${-PI/2}"/>
+    <origin xyz="0 3 1.5" rpy="0 0 ${-PI/2}"/>
     <parent link="world"/>
     <child link="camera_link"/>
@@ -143,5 +143,5 @@
       <origin xyz="0 0 0" rpy="0 0 0"/>
       <geometry>
-	<box size="${camera_link} ${camera_link} ${camera_link}"/>
+	     <box size="${camera_link} ${camera_link} ${camera_link}"/>
       </geometry>
     </collision>
@@ -149,5 +149,5 @@
       <origin xyz="0 0 0" rpy="0 0 0"/>
       <geometry>
-	<box size="${camera_link} ${camera_link} ${camera_link}"/>
+	     <box size="${camera_link} ${camera_link} ${camera_link}"/>
       </geometry>
       <material name="red"/>

File: rrbot_description/urdf/rrbot.xacro (robot description, xacro)
@@ -26,5 +26,5 @@
       <origin xyz="0 0 ${height1/2}" rpy="0 0 0"/>
       <geometry>
-	<box size="${width} ${width} ${height1}"/>
+	     <box size="${width} ${width} ${height1}"/>
       </geometry>
     </collision>
@@ -32,7 +32,7 @@
       <origin xyz="0 0 ${height1/2}" rpy="0 0 0"/>
       <geometry>
-	<box size="${width} ${width} ${height1}"/>
+	     <box size="${width} ${width} ${height1}"/>
       </geometry>
-      <material name="orange"/>
+      <material name="black"/>
     </visual>
     <inertial>
@@ -57,5 +57,5 @@
       <origin xyz="0 0 ${height2/2 - axel_offset}" rpy="0 0 0"/>
       <geometry>
-	<box size="${width} ${width} ${height2}"/>
+	     <box size="${width} ${width} ${height2}"/>
       </geometry>
     </collision>
@@ -63,5 +63,5 @@
       <origin xyz="0 0 ${height2/2 - axel_offset}" rpy="0 0 0"/>
       <geometry>
-	<box size="${width} ${width} ${height2}"/>
+	     <box size="${width} ${width} ${height2}"/>
       </geometry>
       <material name="black"/>
@@ -88,5 +88,5 @@
       <origin xyz="0 0 ${height3/2 - axel_offset}" rpy="0 0 0"/>
       <geometry>
-	<box size="${width} ${width} ${height3}"/>
+	     <box size="${width} ${width} ${height3}"/>
       </geometry>
     </collision>
@@ -94,7 +94,7 @@
       <origin xyz="0 0 ${height3/2 - axel_offset}" rpy="0 0 0"/>
       <geometry>
-	<box size="${width} ${width} ${height3}"/>
+	     <box size="${width} ${width} ${height3}"/>
       </geometry>
-      <material name="orange"/>
+      <material name="black"/>
     </visual>
     <inertial>
@@ -118,5 +118,5 @@
       <origin xyz="0 0 0" rpy="0 0 0"/>
       <geometry>
-	<box size="0.1 0.1 0.1"/>
+	     <box size="0.1 0.1 0.1"/>
       </geometry>
     </collision>
@@ -134,5 +134,5 @@
   </link>
   <joint name="camera_joint" type="fixed">
-    <origin xyz="0 2 1" rpy="0 0 ${-PI/2}"/>
+    <origin xyz="0 3 1.5" rpy="0 0 ${-PI/2}"/>
     <parent link="world"/>
     <child link="camera_link"/>
@@ -143,5 +143,5 @@
       <origin xyz="0 0 0" rpy="0 0 0"/>
       <geometry>
-	<box size="${camera_link} ${camera_link} ${camera_link}"/>
+	     <box size="${camera_link} ${camera_link} ${camera_link}"/>
       </geometry>
     </collision>
@@ -149,5 +149,5 @@
       <origin xyz="0 0 0" rpy="0 0 0"/>
       <geometry>
-	<box size="${camera_link} ${camera_link} ${camera_link}"/>
+	     <box size="${camera_link} ${camera_link} ${camera_link}"/>
       </geometry>
       <material name="red"/>

Commit message: Update broken.xacro to take arguments

File: rrbot_description/urdf/broken.xacro (robot description, xacro)
@@ -2,11 +2,18 @@
 <!-- Revolute-Revolute Manipulator -->
 <robot name="broken" xmlns:xacro="http://www.ros.org/wiki/xacro">
+  <!-- Arguments for tuning dimensions -->
+  <xacro:arg name="d_height1" default="0"/>
+  <xacro:arg name="d_height2" default="0"/>
+  <xacro:arg name="d_height3" default="0"/>
   <!-- Constants for robot dimensions -->
   <xacro:property name="PI" value="3.1415926535897931"/>
   <xacro:property name="mass" value="1" /> <!-- arbitrary value for mass -->
   <xacro:property name="width" value="0.1" /> <!-- Square dimensions (widthxwidth) of beams -->
-  <xacro:property name="height1" value="1.9" /> <!-- Link 1 -->
-  <xacro:property name="height2" value="1" /> <!-- Link 2 -->
-  <xacro:property name="height3" value="1" /> <!-- Link 3 -->
+  <xacro:property name="d_height1" value="$(arg d_height1)" /> <!-- Link 1 -->
+  <xacro:property name="d_height2" value="$(arg d_height2)" /> <!-- Link 2 -->
+  <xacro:property name="d_height3" value="$(arg d_height3)" /> <!-- Link 3 -->
+  <xacro:property name="height1" value="${1.9 + d_height1}" /> <!-- Link 1 -->
+  <xacro:property name="height2" value="${1 + d_height2}" /> <!-- Link 2 -->
+  <xacro:property name="height3" value="${1 + d_height3}" /> <!-- Link 3 -->
   <xacro:property name="camera_link" value="0.05" /> <!-- Size of square 'camera' box -->
   <xacro:property name="axel_offset" value="0.05" /> <!-- Space btw top of beam and the each joint -->
